File: Eagle/rcr_circuit/RCR2.brd (EAGLE design)
At the start: 253.7 x 154.9 mm, 46 parts, among them U1 GY-521MPU6050, X1 RASPI_GPIO_B+_PIN

Commit message: making main board
Parts:
- added 5.6K2: (no value), eagle-ltspice:R1206
- added CONNECTOR2, CONNECTOR3: 2PIN, 2pin_small:2PIN
- added S1: MOMENTARY-SWITCH-SPST-SMD-RIGHT-ANGLE, SparkFun-Switches:TACTILE_SWITCH_SMD_RIGHT_ANGLE
- moved U1 198.3 mm to (224.8, 81.3), flipped to the bottom
- moved U$2 162.9 mm to (229.9, 25.4), flipped to the bottom
- moved U$1 159.6 mm to (203.2, 14.0), flipped to the bottom
- moved D9 121.3 mm to (147.3, 41.9), flipped to the bottom
- moved D1 111.4 mm to (148.6, 87.6), flipped to the bottom
- moved D2 111.4 mm to (148.6, 81.3), flipped to the bottom
- moved D3 111.4 mm to (148.6, 74.9), flipped to the bottom
- moved D4 111.4 mm to (148.6, 68.6), flipped to the bottom
- moved D5 111.4 mm to (148.6, 62.2), flipped to the bottom
- moved D6 111.4 mm to (148.6, 55.9), flipped to the bottom
- moved 10K8 103.4 mm to (69.8, 29.2), flipped to the bottom
- moved 10K1 93.8 mm to (29.2, 15.2), flipped to the bottom
- moved TM1637-SMD1 77.1 mm to (57.1, 68.6), flipped to the bottom, turned to 270 degrees
- moved 10K7 75.2 mm to (27.9, 44.5), flipped to the bottom
- moved X1 71.7 mm to (78.7, 78.7), flipped to the bottom, turned to 180 degrees
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Connections:
- removed net 5V0: X1.2
- removed net GND: U$2.1, X1.6
- removed net GND.2: U$1.J2.4
- removed net VCC: U$2.2
- removed net VCC.2: U$1.J2.3
- new net ACC: 0.1UF5.2, 5.6K2.1, CONNECTOR2.1, D2.C
- new net BATT: CONNECTOR3.1, D9.A
- new net DCDC: 10K5.2, 1M1.2, 4.7UF2.1, D3.C, DMG3415U1.2, DMG3415U2.3
- new net GPIO: 1.8K1.2, 5.6K1.1, D2.A, D6.A, X1.40
- new net N$1: LED1.1, LED2.1, LED3.1, TM1637-SMD1.PIN8
- new net N$10: X1.7
- new net N$103: 100K1.2, 10K3.2, D9.K, DMG3415U2.2
- new net N$104: 10K3.1, 1UF1.1, D5.C, D6.C, S1.2
- new net N$105: 100K1.1, 10K4.2, 1UF1.2, DMG3415U2.1
- new net N$106: 10K4.1, 1UF2.1, 2N7002K1.3
- new net N$107: 2N7002K1.1, D1.C, D4.C
- new net N$108: 0.1UF4.1, 100K2.1, D4.A
- new net N$11: LED1.8, LED2.8, LED3.8, TM1637-SMD1.PIN4
- new net N$110: 100K2.2, 100K3.1, 4.7UF2.2
- new net N$111: 100K4.2, 5.6K1.2, DMG3415U1.3
- new net N$112: X1.29
- new net N$113: 100K3.2, 100K4.1, D5.A
- new net N$115: 0.1UF5.1, 100K5.1, D1.A
- new net N$116: 1M1.1, D3.A, DMG3415U1.1
- new net N$117: 10K6.1, 22UF1.1, 2N7002K2.3
- new net N$118: 2N7002K2.1, 3.3K1.2, 5.6K2.2
- new net N$12: LED1.9, LED2.9, LED3.9, TM1637-SMD1.PIN3
- new net N$13: LED3.5, TM1637-SMD1.PIN10
- new net N$133: X1.32
- new net N$134: X1.33
- new net N$14: LED3.10, TM1637-SMD1.PIN11
- new net N$15: LED2.5, TM1637-SMD1.PIN12
- new net N$16: LED2.10, TM1637-SMD1.PIN13
- new net N$17: LED1.5, TM1637-SMD1.PIN14
- new net N$18: LED1.10, TM1637-SMD1.PIN15
- new net N$19: 0.1UF1.1, 10K2.1, 10K8.1, TM1637-SMD1.PIN18
- new net N$2: LED1.2, LED2.2, LED3.2, TM1637-SMD1.PIN9
- new net N$20: 0.1UF2.1, 10K1.1, 10K7.1, TM1637-SMD1.PIN17
- new net N$21: 0.1UF3.1, 10K1.2, 10K2.2, 10K7.2, 10K8.2, 4.7UF1.1, TM1637-SMD1.PIN16
- new net N$22: 0.1UF1.2, 0.1UF2.2, 0.1UF3.2, 4.7UF1.2, TM1637-SMD1.PIN1
- new net N$3: LED1.3, LED2.3, LED3.3, TM1637-SMD1.PIN2
- new net N$34: U$1.J2.1, U$2.3, U1.SCL, X1.5
- new net N$4: X1.11
- new net N$44: 0.1UF4.2, 1.8K1.1, 100K5.2, 10K5.1, 1UF2.2, 22UF1.2, 2N7002K1.2, 2N7002K2.2, 3.3K1.1, CONNECTOR2.2, CONNECTOR3.2, S1.1, U$1.J2.4, U$2.1, U1.GND, X1.6
- new net N$5: X1.12
- new net N$6: LED1.4, LED2.4, LED3.4, TM1637-SMD1.PIN7
- new net N$61: X1.13
- new net N$62: X1.15
- new net N$68: U$1.J2.2, U$2.4, U1.SDA, X1.3
- new net N$7: X1.22
- new net N$8: LED1.6, LED2.6, LED3.6, TM1637-SMD1.PIN5
- new net N$81: X1.31
- new net N$9: LED1.7, LED2.7, LED3.7, TM1637-SMD1.PIN6
- new net N$98: X1.16
- new net N$99: X1.18
- new net VDD: U$1.J2.3, U$2.2, U1.VCC, X1.2
Other:
- board size 253.7 x 154.9 mm -> 140 x 83 mm
