File: Eagle/rcr_circuit/RCR2.sch (EAGLE design)
At the start: 46 parts, among them U1 GY-521MPU6050, X1 RASPI_GPIO_B+_PIN

Commit message: making main board
Parts:
- added 5.6K2: (no value), eagle-ltspice:RR1206
- added CONNECTOR2, CONNECTOR3: 2PIN, 2pin_small:2PIN
- added S1: MOMENTARY-SWITCH-SPST-SMD-RIGHT-ANGLE, SparkFun-Switches:MOMENTARY-SWITCH-SPST-SMD-RIGHT-ANGLE
Connections:
- new net ACC: 0.1UF5.2, 5.6K2.1, CONNECTOR2.1, D2.C
- new net BATT: CONNECTOR3.1, D9.A
- new net DCDC: 10K5.2, 1M1.2, 4.7UF2.1, D3.C, DMG3415U1.E, DMG3415U2.C
- new net GPIO: 1.8K1.2, 5.6K1.1, D2.A, D6.A, X1.GPIO21
- new net N$1: LED1.1, LED2.1, LED3.1, TM1637-SMD1.P$8
- new net N$10: X1.GPIO04
- new net N$103: 100K1.2, 10K3.2, D9.C, DMG3415U2.E
- new net N$104: 10K3.1, 1UF1.1, D5.C, D6.C, S1.2
- new net N$105: 100K1.1, 10K4.2, 1UF1.2, DMG3415U2.B
- new net N$106: 10K4.1, 1UF2.1, 2N7002K1.C
- new net N$107: 2N7002K1.B, D1.C, D4.C
- new net N$108: 0.1UF4.1, 100K2.1, D4.A
- new net N$11: LED1.8, LED2.8, LED3.8, TM1637-SMD1.P$4
- new net N$110: 100K2.2, 100K3.1, 4.7UF2.2
- new net N$111: 100K4.2, 5.6K1.2, DMG3415U1.C
- new net N$112: X1.GPIO05
- new net N$113: 100K3.2, 100K4.1, D5.A
- new net N$115: 0.1UF5.1, 100K5.1, D1.A
- new net N$116: 1M1.1, D3.A, DMG3415U1.B
- new net N$117: 10K6.1, 22UF1.1, 2N7002K2.C
- new net N$118: 2N7002K2.B, 3.3K1.2, 5.6K2.2
- new net N$12: LED1.9, LED2.9, LED3.9, TM1637-SMD1.P$3
- new net N$13: LED3.5, TM1637-SMD1.P$10
- new net N$133: X1.GPIO12
- new net N$134: X1.GPIO13
- new net N$14: LED3.10, TM1637-SMD1.P$11
- new net N$15: LED2.5, TM1637-SMD1.P$12
- new net N$16: LED2.10, TM1637-SMD1.P$13
- new net N$17: LED1.5, TM1637-SMD1.P$14
- new net N$18: LED1.10, TM1637-SMD1.P$15
- new net N$19: 0.1UF1.1, 10K2.1, 10K8.1, TM1637-SMD1.P$18
- new net N$2: LED1.2, LED2.2, LED3.2, TM1637-SMD1.P$9
- new net N$20: 0.1UF2.1, 10K1.1, 10K7.1, TM1637-SMD1.P$17
- new net N$21: 0.1UF3.1, 10K1.2, 10K2.2, 10K7.2, 10K8.2, 4.7UF1.1, TM1637-SMD1.P$16
- new net N$22: 0.1UF1.2, 0.1UF2.2, 0.1UF3.2, 4.7UF1.2, TM1637-SMD1.P$1
- new net N$3: LED1.3, LED2.3, LED3.3, TM1637-SMD1.P$2
- new net N$34: U$1.SCL.2, U$2.SCL, U1.SCL, X1.SCL
- new net N$4: X1.GPIO17
- new net N$44: 0.1UF4.2, 1.8K1.1, 100K5.2, 10K5.1, 1UF2.2, 22UF1.2, 2N7002K1.E, 2N7002K2.E, 3.3K1.1, CONNECTOR2.2, CONNECTOR3.2, S1.1, U$1.GND.2, U$2.GND, U1.GND, X1.GND
- new net N$5: X1.GPIO18
- new net N$6: LED1.4, LED2.4, LED3.4, TM1637-SMD1.P$7
- new net N$61: X1.GPIO27
- new net N$62: X1.GPIO22
- new net N$68: U$1.SDA.2, U$2.SDA, U1.SDA, X1.SDA
- new net N$7: X1.GPIO25
- new net N$8: LED1.6, LED2.6, LED3.6, TM1637-SMD1.P$5
- new net N$81: X1.GPIO06
- new net N$9: LED1.7, LED2.7, LED3.7, TM1637-SMD1.P$6
- new net N$98: X1.GPIO23
- new net N$99: X1.GPIO24
- new net VDD: U$1.VCC.2, U$2.VCC, U1.VCC, X1.5V0
Other:
- moved on the sheet: 0.1UF1, 0.1UF2, 0.1UF3, 0.1UF4, 0.1UF5, 1.8K1, 100K1, 100K2, 100K3, 100K4, 100K5, 10K1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
