File: Eagle/ups_unit/ups_unit.sch (EAGLE design)
At the start: 36 parts

Commit message: RPi UPS unit
Parts:
- removed S1: MOMENTARY-SWITCH-SPST-SMD-RIGHT-ANGLE, SparkFun-Switches:MOMENTARY-SWITCH-SPST-SMD-RIGHT-ANGLE
- added POWER　SWITCH: (no value), pinhead:PINHD-1X2
- renumbered JP1 to GPIO, JP2 to DCDC, JP3 to BATT, JP4 to ACC
Connections:
- net GND: now also POWER　SWITCH.2; no longer S1.1
- net N$104: now also POWER　SWITCH.1; no longer S1.2
- net N$116: now also 10K6.2
Changed lines of the file:
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@@
 <setting verticaltext="up"/>
 </settings>
-<grid distance="1.27" unitdist="mm" unit="mm" style="lines" multiple="1" display="yes" altdistance="0.01" altunitdist="inch" altunit="inch"/>
+<grid distance="0.1" unitdist="inch" unit="inch" style="lines" multiple="1" display="no" altdistance="0.01" altunitdist="inch" altunit="inch"/>
 <layers>
 <layer number="1" name="Top" color="4" fill="1" visible="no" active="no"/>
@@
 </variantdefs>
 <classes>
-<class number="0" name="default" width="0" drill="0">
+<class number="0" name="default" width="0.4" drill="0.3">
+<clearance class="0" value="0.3"/>
 </class>
 </classes>
@@
 <part name="D9" library="diode" library_urn="urn:adsk.eagle:library:210" deviceset="GF1" device="" package3d_urn="urn:adsk.eagle:package:43452/2"/>
 <part name="5.6K2" library="eagle-ltspice" library_urn="urn:adsk.eagle:library:217" deviceset="R" device="R1206" package3d_urn="urn:adsk.eagle:package:13301/1"/>
-<part name="S1" library="SparkFun-Switches" deviceset="MOMENTARY-SWITCH-SPST" device="-SMD-RIGHT-ANGLE"/>
-<part name="JP1" library="pinhead" library_urn="urn:adsk.eagle:library:325" deviceset="PINHD-1X2" device="" package3d_urn="urn:adsk.eagle:package:22435/2"/>
-<part name="JP2" library="pinhead" library_urn="urn:adsk.eagle:library:325" deviceset="PINHD-1X2" device="" package3d_urn="urn:adsk.eagle:package:22435/2"/>
-<part name="JP3" library="pinhead" library_urn="urn:adsk.eagle:library:325" deviceset="PINHD-1X2" device="" package3d_urn="urn:adsk.eagle:package:22435/2"/>
-<part name="JP4" library="pinhead" library_urn="urn:adsk.eagle:library:325" deviceset="PINHD-1X2" device="" package3d_urn="urn:adsk.eagle:package:22435/2"/>
+<part name="GPIO" library="pinhead" library_urn="urn:adsk.eagle:library:325" deviceset="PINHD-1X2" device="" package3d_urn="urn:adsk.eagle:package:22435/2"/>
+<part name="DCDC" library="pinhead" library_urn="urn:adsk.eagle:library:325" deviceset="PINHD-1X2" device="" package3d_urn="urn:adsk.eagle:package:22435/2"/>
+<part name="BATT" library="pinhead" library_urn="urn:adsk.eagle:library:325" deviceset="PINHD-1X2" device="" package3d_urn="urn:adsk.eagle:package:22435/2"/>
+<part name="ACC" library="pinhead" library_urn="urn:adsk.eagle:library:325" deviceset="PINHD-1X2" device="" package3d_urn="urn:adsk.eagle:package:22435/2"/>
+<part name="POWER　SWITCH" library="pinhead" library_urn="urn:adsk.eagle:library:325" deviceset="PINHD-1X2" device="" package3d_urn="urn:adsk.eagle:package:22435/2"/>
 </parts>
 <sheets>
@@
 <attribute name="VALUE" x="183.642" y="27.94" size="1.778" layer="96" rot="R90"/>
 </instance>
-<instance part="S1" gate="G$1" x="33.02" y="-2.54" smashed="yes" rot="R90">
-<attribute name="NAME" x="31.496" y="-2.54" size="1.778" layer="95" font="vector" rot="R90" align="bottom-center"/>
-<attribute name="VALUE" x="33.528" y="-2.54" size="1.778" layer="96" font="vector" rot="R90" align="top-center"/>
-</instance>
-<instance part="JP1" gate="G$1" x="201.93" y="8.89" smashed="yes">
+<instance part="GPIO" gate="G$1" x="201.93" y="8.89" smashed="yes">
 <attribute name="NAME" x="195.58" y="14.605" size="1.778" layer="95"/>
 <attribute name="VALUE" x="195.58" y="3.81" size="1.778" layer="96"/>
 </instance>
-<instance part="JP2" gate="G$1" x="201.93" y="68.58" smashed="yes">
+<instance part="DCDC" gate="G$1" x="201.93" y="68.58" smashed="yes">
 <attribute name="NAME" x="195.58" y="74.295" size="1.778" layer="95"/>
 <attribute name="VALUE" x="195.58" y="63.5" size="1.778" layer="96"/>
 </instance>
-<instance part="JP3" gate="G$1" x="1.27" y="15.24" smashed="yes" rot="R180">
+<instance part="BATT" gate="G$1" x="1.27" y="15.24" smashed="yes" rot="R180">
 <attribute name="NAME" x="2.54" y="20.955" size="1.778" layer="95" rot="R180"/>
 <attribute name="VALUE" x="7.62" y="20.32" size="1.778" layer="96" rot="R180"/>
 </instance>
-<instance part="JP4" gate="G$1" x="1.27" y="6.35" smashed="yes" rot="R180">
+<instance part="ACC" gate="G$1" x="1.27" y="6.35" smashed="yes" rot="R180">
 <attribute name="NAME" x="2.54" y="-0.635" size="1.778" layer="95" rot="R180"/>
 <attribute name="VALUE" x="7.62" y="11.43" size="1.778" layer="96" rot="R180"/>
+</instance>
+<instance part="POWER　SWITCH" gate="G$1" x="40.64" y="-3.81" smashed="yes">
+<attribute name="NAME" x="34.29" y="1.905" size="1.778" layer="95"/>
+<attribute name="VALUE" x="34.29" y="-8.89" size="1.778" layer="96"/>
 </instance>
 </instances>
@@
 <wire x1="33.02" y1="54.61" x2="33.02" y2="11.43" width="0.1524" layer="91"/>
 <junction x="33.02" y="54.61"/>
-<wire x1="33.02" y1="11.43" x2="33.02" y2="2.54" width="0.1524" layer="91"/>
+<wire x1="33.02" y1="11.43" x2="33.02" y2="-1.27" width="0.1524" layer="91"/>
 <junction x="33.02" y="11.43"/>
-<pinref part="S1" gate="G$1" pin="2"/>
+<pinref part="POWER　SWITCH" gate="G$1" pin="1"/>
+<wire x1="38.1" y1="-1.27" x2="33.02" y2="-1.27" width="0.1524" layer="91"/>
+<label x="41.91" y="-1.27" size="1.778" layer="95"/>
 </segment>
 </net>
@@
 <junction x="127" y="71.12"/>
 <label x="165.1" y="73.66" size="1.778" layer="95"/>
-<pinref part="JP2" gate="G$1" pin="1"/>
+<pinref part="DCDC" gate="G$1" pin="1"/>
 <wire x1="151.13" y1="71.12" x2="199.39" y2="71.12" width="0.1524" layer="91"/>
 </segment>
@@
 <junction x="146.05" y="16.51"/>
 <label x="187.96" y="12.7" size="1.778" layer="95"/>
-<pinref part="JP1" gate="G$1" pin="1"/>
+<pinref part="GPIO" gate="G$1" pin="1"/>
 <wire x1="146.05" y1="11.43" x2="199.39" y2="11.43" width="0.1524" layer="91"/>
 <junction x="146.05" y="11.43"/>
@@
 <pinref part="D3" gate="G$1" pin="A"/>
 <wire x1="139.7" y1="57.15" x2="139.7" y2="60.96" width="0.1524" layer="91"/>
-<pinref part="1M1" gate="G$1" pin="1"/>
-<wire x1="139.7" y1="57.15" x2="151.13" y2="57.15" width="0.1524" layer="91"/>
-<wire x1="151.13" y1="57.15" x2="151.13" y2="58.42" width="0.1524" layer="91"/>
 <pinref part="DMG3415U1" gate="D" pin="B"/>
 <wire x1="132.08" y1="57.15" x2="139.7" y2="57.15" width="0.1524" layer="91"/>
 <junction x="139.7" y="57.15"/>
-</segment>
-</net>
-<net name="N$117" class="0">
-<segment>
-<pinref part="10K6" gate="G$1" pin="1"/>
-<pinref part="22UF1" gate="G$1" pin="1"/>
-<wire x1="151.13" y1="45.72" x2="151.13" y2="44.45" width="0.1524" layer="91"/>
-<pinref part="2N7002K2" gate="G$1" pin="C"/>
-<wire x1="151.13" y1="44.45" x2="151.13" y2="41.91" width="0.1524" layer="91"/>
-<wire x1="151.13" y1="44.45" x2="160.02" y2="44.45" width="0.1524" layer="91"/>
-<wire x1="160.02" y1="44.45" x2="160.02" y2="43.18" width="0.1524" layer="91"/>
-<junction x="151.13" y="44.45"/>
+<pinref part="1M1" gate="G$1" pin="1"/>
+<pinref part="10K6" gate="G$1" pin="2"/>
+<wire x1="151.13" y1="58.42" x2="151.13" y2="55.88" width="0.1524" layer="91"/>
+<wire x1="139.7" y1="57.15" x2="139.7" y2="55.88" width="0.1524" layer="91"/>
+<wire x1="139.7" y1="55.88" x2="151.13" y2="55.88" width="0.1524" layer="91"/>
+<junction x="151.13" y="55.88"/>
+<wire x1="151.13" y1="55.88" x2="151.13" y2="54.61" width="0.1524" layer="91"/>
 </segment>
 </net>
@@
 <junction x="85.09" y="6.35"/>
 <label x="15.24" y="7.62" size="1.778" layer="95"/>
-<pinref part="JP4" gate="G$1" pin="2"/>
+<pinref part="ACC" gate="G$1" pin="2"/>
 </segment>
 </net>
@@
 <label x="8.89" y="16.51" size="1.778" layer="95"/>
 <wire x1="3.81" y1="15.24" x2="21.59" y2="15.24" width="0.1524" layer="91"/>
-<pinref part="JP3" gate="G$1" pin="2"/>
+<pinref part="BATT" gate="G$1" pin="2"/>
 </segment>
 </net>
@@
 <junction x="64.77" y="-11.43"/>
 <wire x1="33.02" y1="-11.43" x2="64.77" y2="-11.43" width="0.1524" layer="91"/>
-<pinref part="S1" gate="G$1" pin="1"/>
-<wire x1="33.02" y1="-7.62" x2="33.02" y2="-11.43" width="0.1524" layer="91"/>
 <junction x="33.02" y="-11.43"/>
 <wire x1="12.7" y1="12.7" x2="12.7" y2="3.81" width="0.1524" layer="91"/>
@@
 <wire x1="21.59" y1="-11.43" x2="33.02" y2="-11.43" width="0.1524" layer="91"/>
 <label x="8.89" y="1.27" size="1.778" layer="95"/>
-<pinref part="JP1" gate="G$1" pin="2"/>
+<pinref part="GPIO" gate="G$1" pin="2"/>
 <wire x1="199.39" y1="8.89" x2="186.69" y2="8.89" width="0.1524" layer="91"/>
 <wire x1="186.69" y1="8.89" x2="186.69" y2="-11.43" width="0.1524" layer="91"/>
 <wire x1="186.69" y1="-11.43" x2="151.13" y2="-11.43" width="0.1524" layer="91"/>
 <junction x="151.13" y="-11.43"/>
-<pinref part="JP2" gate="G$1" pin="2"/>
+<pinref part="DCDC" gate="G$1" pin="2"/>
 <wire x1="186.69" y1="8.89" x2="186.69" y2="68.58" width="0.1524" layer="91"/>
 <wire x1="186.69" y1="68.58" x2="199.39" y2="68.58" width="0.1524" layer="91"/>
 <junction x="186.69" y="8.89"/>
-<pinref part="JP3" gate="G$1" pin="1"/>
+<pinref part="BATT" gate="G$1" pin="1"/>
 <wire x1="12.7" y1="12.7" x2="3.81" y2="12.7" width="0.1524" layer="91"/>
-<pinref part="JP4" gate="G$1" pin="1"/>
+<pinref part="ACC" gate="G$1" pin="1"/>
 <wire x1="12.7" y1="3.81" x2="3.81" y2="3.81" width="0.1524" layer="91"/>
-</segment>
-</net>
+<pinref part="POWER　SWITCH" gate="G$1" pin="2"/>
+<wire x1="38.1" y1="-3.81" x2="33.02" y2="-3.81" width="0.1524" layer="91"/>
+<wire x1="33.02" y1="-3.81" x2="33.02" y2="-11.43" width="0.1524" layer="91"/>
+<label x="41.91" y="-6.35" size="1.778" layer="95"/>
+</segment>
+</net>
+<net name="N$1" class="0">
+<segment>
+<pinref part="22UF1" gate="G$1" pin="1"/>
+<pinref part="2N7002K2" gate="G$1" pin="C"/>
+<wire x1="160.02" y1="44.45" x2="160.02" y2="43.18" width="0.1524" layer="91"/>
+<pinref part="10K6" gate="G$1" pin="1"/>
+<wire x1="151.13" y1="45.72" x2="151.13" y2="44.45" width="0.1524" layer="91"/>
+<wire x1="151.13" y1="44.45" x2="160.02" y2="44.45" width="0.1524" layer="91"/>
+<junction x="151.13" y="44.45"/>
+<wire x1="151.13" y1="44.45" x2="151.13" y2="41.91" width="0.1524" layer="91"/>
+</segment>
+</net>
