File: gpio_unit/gpio_unit.brd (EAGLE design)
At the start: 89.2 x 39.4 mm, 18 parts, among them X1 RASPI_GPIO_B+_PIN

Commit message: arrange comment
Parts:
- renumbered JP2 to I2CPORT_1, JP3 to I2CPORT_2, JP4 to I2CPORT_3, SV1 to 7SEG_1, SV10 to MPU6050, SV2 to 7SEG_2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
